File: Esquematico/Central/central/central.kicad_sch (KiCad schematic)
At the start: 23 parts, among them J1 Conn_01x03_Socket, J2 Conn_01x03_Socket, J3 Conn_01x03_Socket, J4 Conn_01x03_Socket, J5 USB_A, K1 JQC-3FF-005-1Z, K2 JQC-3FF-005-1Z, K3 JQC-3FF-005-1Z, Q1 2TY, Q2 2TY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

Commit message: Commit automático
Parts:
- removed J5: USB_A, Connector_USB:USB_A_Stewart_SS-52100-001_Horizontal, symbol Connector:USB_A
- removed U2: AMS1117-3.3, Package_TO_SOT_SMD:SOT-89-3_Handsoldering, symbol Regulator_Linear:AMS1117-3.3
- added C2, C3: 100n, Capacitor_SMD:C_1206_3216Metric_Pad1.33x1.80mm_HandSolder, symbol Device:C
- added J5, J6, J7, J8: Conn_01x01_Pin, Connector_PinHeader_1.00mm:PinHeader_1x01_P1.00mm_Vertical, symbol Connector:Conn_01x01_Pin
- added R4: 470R, Resistor_THT:R_Axial_DIN0309_L9.0mm_D3.2mm_P12.70mm_Horizontal, symbol Device:R
- added R5: 100R, Resistor_THT:R_Axial_DIN0309_L9.0mm_D3.2mm_P12.70mm_Horizontal, symbol Device:R
- added U3: EL817, Package_SO:SOP-4_3.8x4.1mm_P2.54mm, symbol Isolator:EL817
- R1, R2, R3: value 242 -> 2K
Connections:
- net GND: now also J4.1 (Pin_1), C2.2, C3.2, J6.1 (Pin_1), J8.1 (Pin_1), U3.3; no longer J4.3 (Pin_3)
- net VCC: now also C3.1, J7.1 (Pin_1); no longer C1.1, Q1.1 (E), Q2.1 (E), Q3.1 (E)
- net at U1.10 (GPIO17/U1TXD/ADC2_CH6): now also Brd1.3 (SCL); no longer Brd1.4 (SDA)
- net at U1.11 (GPIO18/U1RXD/ADC2_CH7/CLK_OUT3): now also Brd1.4 (SDA); no longer Brd1.3 (SCL)
- net at U1.13 (GPIO19/U1RTS/ADC2_CH8/CLK_OUT2/USB_D-): now also BZ1.2 (-)
- net at U1.38 (GPIO2/TOUCH2/ADC1_CH1): now also R5.2; no longer J4.1 (Pin_1)
- net at U1.39 (GPIO1/TOUCH1/ADC1_CH0): no longer BZ1.2 (-)
- new net: R5.1, U3.4
- new net: R4.2, U3.1
- new net: J4.3 (Pin_3), U3.2
- new net +5V: C1.1, C2.1, J5.1 (Pin_1), Q1.1 (E), Q2.1 (E), Q3.1 (E), R4.1
Other:
- moved on the sheet: BZ1, Brd1, J4
